Commit message: bottom and top arm

File: assignment4/urdf/lynxmotion.urdf.xacro (robot description, xacro)
@@ -21,16 +21,20 @@
 				<box size="0.4 0.1 0.2"/>
 			</geometry>
-			<origin rpy="0 1.57075 0" xyz="0 0 -0.25"/>
+			<origin rpy="0 1.57075 0" xyz="0 0 0.2"/>
 		</visual>
 	</link>
-	<joint name="base_to_bottom_arm" type="fixed">
+	<joint name="base_to_bottom_arm" type="revolute">
+		<axis xyz="0 0 1"/>
+		<limit effort="1000.0" lower="-1.548" upper="1.548" velocity="0.5"/>
+		<origin xyz="0 0 0.65"/>
 		<parent link="base_link"/>
 		<child link="bottom_arm"/>
-		<origin xyz="0 0 0.65"/>
 	</joint>
-	<joint name="bottom_to_top_arm" type="fixed">
+	<joint name="bottom_to_top_arm" type="revolute">
+		<axis xyz="0 1 0"/>
+		<limit effort="1000.0" lower="-1.548" upper="1.548" velocity="0.5"/>
+		<origin xyz="0 0 0"/>
 		<parent link="bottom_arm"/>
 		<child link="top_arm"/>
-		<origin xyz="0 0 0.4"/>
 	</joint>
 </robot>

Commit message: help notes for getting started

File: assignment4/urdf/lynxmotion.urdf.xacro (robot description, xacro)
@@ -1,4 +1,7 @@
 <?xml version="1.0"?>
 	<robot name="lynxmotion">
+		<material name="blue">
+			<color rgba="0 0 0.8 1"/>
+		</material>
 		<link name="base_link">
 		<visual>
@@ -6,4 +9,5 @@
 				<cylinder length="0.4" radius="0.3"/>
 			</geometry>
+			<origin rpy="0 0 0" xyz="0 0 -0.25"/>
 		</visual>
 	</link>
@@ -13,4 +17,5 @@
 				<box size="0.4 0.1 0.2"/>
 			</geometry>
+			<material name="blue"/>
 			<origin rpy="0 1.57075 0" xyz="0 0 -0.25"/>
 		</visual>

Commit message: Changed velociy be come XACRO parametter

File: assignment4/urdf/lynxmotion.urdf.xacro (robot description, xacro)
@@ -1,4 +1,5 @@
 <?xml version="1.0"?>
-	<robot name="lynxmotion">
+	<robot name="lynxmotion" xmlns:xacro="http://ros.org/wiki/xacro">
+	<xacro:property name="velocity" value="0.5"/>
 	<material name="blue">
 		<color rgba="0 0 0.8 1"/>
@@ -66,5 +67,5 @@
 	<joint name="left_gripper_joint" type="revolute">
 		<axis xyz="0 1 0"/>
-		<limit effort="1000.0" lower="-1.57075" upper="0" velocity="0.5"/>
+		<limit effort="1000.0" lower="-1.57075" upper="0" velocity="${velocity}"/>
 		<origin rpy="0 0 0" xyz="0 0 0.2"/>
 		<parent link="wrist"/>
@@ -73,5 +74,5 @@
 	<joint name="right_gripper_joint" type="revolute">
 		<axis xyz="0 0 -1"/>
-		<limit effort="1000.0" lower="0.0" upper="0.548" velocity="0.5"/>
+		<limit effort="1000.0" lower="0.0" upper="0.548" velocity="${velocity}"/>
 		<origin rpy="0 0 0" xyz="0 0 0.2"/>
 		<parent link="wrist"/>
@@ -80,5 +81,5 @@
 	<joint name="base_block_to_base_link" type="revolute">
 		<axis xyz="0 0 1"/>
-		<limit effort="1000.0" lower="-1.548" upper="1.548" velocity="0.5"/>
+		<limit effort="1000.0" lower="-1.548" upper="1.548" velocity="${velocity}"/>
 		<origin xyz="0 0 0.1"/>
 		<parent link="base_link"/>
@@ -87,5 +88,5 @@
 	<joint name="base_to_bottom_arm" type="revolute">
 		<axis xyz="0 1 0"/>
-		<limit effort="1000.0" lower="-1.548" upper="1.548" velocity="0.5"/>
+		<limit effort="1000.0" lower="-1.548" upper="1.548" velocity="${velocity}"/>
 		<origin xyz="0 0 0.2"/>
 		<parent link="base_rotate"/>
@@ -94,5 +95,5 @@
 	<joint name="bottom_to_top_arm" type="revolute">
 		<axis xyz="0 1 0"/>
-		<limit effort="1000.0" lower="-1.548" upper="1.548" velocity="0.5"/>
+		<limit effort="1000.0" lower="-1.548" upper="1.548" velocity="${velocity}"/>
 		<origin xyz="0 0 0.4"/>
 		<parent link="bottom_arm"/>
@@ -101,5 +102,5 @@
 	<joint name="wrist_rotate" type="revolute">
 		<axis xyz="0 0 1"/>
-		<limit effort="1000.0" lower="-1.548" upper="1.548" velocity="0.5"/>
+		<limit effort="1000.0" lower="-1.548" upper="1.548" velocity="${velocity}"/>
 		<origin xyz="0 0 0.4"/>
 		<parent link="top_arm"/>

Commit message: Changed velociy be come XACRO parametter (reverted from commit 54ef8c7e565d71022b5a948bfccd5d9764c27912)

File: assignment4/urdf/lynxmotion.urdf.xacro (robot description, xacro)
@@ -1,5 +1,4 @@
 <?xml version="1.0"?>
-	<robot name="lynxmotion" xmlns:xacro="http://ros.org/wiki/xacro">
-	<xacro:property name="velocity" value="0.5"/>
+	<robot name="lynxmotion">
 	<material name="blue">
 		<color rgba="0 0 0.8 1"/>
@@ -67,5 +66,5 @@
 	<joint name="left_gripper_joint" type="revolute">
 		<axis xyz="0 1 0"/>
-		<limit effort="1000.0" lower="-1.57075" upper="0" velocity="${velocity}"/>
+		<limit effort="1000.0" lower="-1.57075" upper="0" velocity="0.5"/>
 		<origin rpy="0 0 0" xyz="0 0 0.2"/>
 		<parent link="wrist"/>
@@ -74,5 +73,5 @@
 	<joint name="right_gripper_joint" type="revolute">
 		<axis xyz="0 0 -1"/>
-		<limit effort="1000.0" lower="0.0" upper="0.548" velocity="${velocity}"/>
+		<limit effort="1000.0" lower="0.0" upper="0.548" velocity="0.5"/>
 		<origin rpy="0 0 0" xyz="0 0 0.2"/>
 		<parent link="wrist"/>
@@ -81,5 +80,5 @@
 	<joint name="base_block_to_base_link" type="revolute">
 		<axis xyz="0 0 1"/>
-		<limit effort="1000.0" lower="-1.548" upper="1.548" velocity="${velocity}"/>
+		<limit effort="1000.0" lower="-1.548" upper="1.548" velocity="0.5"/>
 		<origin xyz="0 0 0.1"/>
 		<parent link="base_link"/>
@@ -88,5 +87,5 @@
 	<joint name="base_to_bottom_arm" type="revolute">
 		<axis xyz="0 1 0"/>
-		<limit effort="1000.0" lower="-1.548" upper="1.548" velocity="${velocity}"/>
+		<limit effort="1000.0" lower="-1.548" upper="1.548" velocity="0.5"/>
 		<origin xyz="0 0 0.2"/>
 		<parent link="base_rotate"/>
@@ -95,5 +94,5 @@
 	<joint name="bottom_to_top_arm" type="revolute">
 		<axis xyz="0 1 0"/>
-		<limit effort="1000.0" lower="-1.548" upper="1.548" velocity="${velocity}"/>
+		<limit effort="1000.0" lower="-1.548" upper="1.548" velocity="0.5"/>
 		<origin xyz="0 0 0.4"/>
 		<parent link="bottom_arm"/>
@@ -102,5 +101,5 @@
 	<joint name="wrist_rotate" type="revolute">
 		<axis xyz="0 0 1"/>
-		<limit effort="1000.0" lower="-1.548" upper="1.548" velocity="${velocity}"/>
+		<limit effort="1000.0" lower="-1.548" upper="1.548" velocity="0.5"/>
 		<origin xyz="0 0 0.4"/>
 		<parent link="top_arm"/>
