Commit message: calibrating arms

File: assignment4/urdf/lynxmotion.urdf (robot description, URDF)
Before this commit: robot lynxmotion, 3 links, 2 joints
Joints:
- joint base_to_bottom_arm: origin xyz=0 0 0.65 -> xyz=0 0 0.4
- joint bottom_to_top_arm: origin xyz=0 0 0 -> xyz=0 0 0.3

File: assignment4/urdf/lynxmotion.urdf.xacro (robot description, xacro)
@@ -9,5 +9,5 @@
 				<cylinder length="0.4" radius="0.3"/>
 			</geometry>
-			<origin rpy="0 0 0" xyz="0 0 -0.25"/>
+			<origin rpy="0 0 0" xyz="0 0 0.2"/>
 		</visual>
 	</link>
@@ -18,5 +18,5 @@
 			</geometry>
 			<material name="blue"/>
-			<origin rpy="0 1.57075 0" xyz="0 0 -0.25"/>
+			<origin rpy="0 1.57075 0" xyz="0 0 0.15"/>
 		</visual>
 	</link>
@@ -26,5 +26,5 @@
 				<box size="0.4 0.1 0.2"/>
 			</geometry>
-			<origin rpy="0 1.57075 0" xyz="0 0 0.2"/>
+			<origin rpy="0 1.57075 0" xyz="0 0 0.3"/>
 		</visual>
 	</link>
@@ -32,5 +32,5 @@
 		<axis xyz="0 0 1"/>
 		<limit effort="1000.0" lower="-1.548" upper="1.548" velocity="0.5"/>
-		<origin xyz="0 0 0.65"/>
+		<origin xyz="0 0 0.4"/>
 		<parent link="base_link"/>
 		<child link="bottom_arm"/>
@@ -39,5 +39,5 @@
 		<axis xyz="0 1 0"/>
 		<limit effort="1000.0" lower="-1.548" upper="1.548" velocity="0.5"/>
-		<origin xyz="0 0 0"/>
+		<origin xyz="0 0 0.3"/>
 		<parent link="bottom_arm"/>
 		<child link="top_arm"/>

Commit message: debugging base block and base link

File: assignment4/urdf/lynxmotion.urdf (robot description, URDF)
Before this commit: robot lynxmotion, 3 links, 2 joints
Links:
- added link base_block; visual cylinder length=0.2 radius=0.3
- link base_link: geometry visual cylinder length=0.2 radius=0.1
Joints:
- added joint base_block_to_base_link: type revolute, parent base_block, child base_link, origin xyz=0 0 0.4, axis 0 0 1, limit lower=-1.548 upper=1.548 effort=1000.0 velocity=0.5
- joint base_to_bottom_arm: axis 0 0 1 -> 0 1 0; origin xyz=0 0 0.4 -> xyz=0 0 0.5

File: assignment4/urdf/lynxmotion.urdf.xacro (robot description, xacro)
@@ -1,13 +1,21 @@
 <?xml version="1.0"?>
 	<robot name="lynxmotion">
-		<material name="blue">
-			<color rgba="0 0 0.8 1"/>
-		</material>
-		<link name="base_link">
+	<material name="blue">
+		<color rgba="0 0 0.8 1"/>
+	</material>
+	<link name="base_block">
 		<visual>
 			<geometry>
-				<cylinder length="0.4" radius="0.3"/>
+				<cylinder length="0.2" radius="0.3"/>
 			</geometry>
-			<origin rpy="0 0 0" xyz="0 0 0.2"/>
+			<origin rpy="0 0 0" xyz="0 0 0.3"/>
+		</visual>
+	</link>
+	<link name="base_link">
+		<visual>
+			<geometry>
+				<cylinder length="0.2" radius="0.1"/>
+			</geometry>
+			<origin rpy="0 0 0" xyz="0 0 0.3"/>
 		</visual>
 	</link>
@@ -29,8 +37,15 @@
 		</visual>
 	</link>
-	<joint name="base_to_bottom_arm" type="revolute">
+	<joint name="base_block_to_base_link" type="revolute">
 		<axis xyz="0 0 1"/>
 		<limit effort="1000.0" lower="-1.548" upper="1.548" velocity="0.5"/>
 		<origin xyz="0 0 0.4"/>
+		<parent link="base_block"/>
+		<child link="base_link"/>
+	</joint>
+	<joint name="base_to_bottom_arm" type="revolute">
+		<axis xyz="0 1 0"/>
+		<limit effort="1000.0" lower="-1.548" upper="1.548" velocity="0.5"/>
+		<origin xyz="0 0 0.5"/>
 		<parent link="base_link"/>
 		<child link="bottom_arm"/>

Commit message: gripper and wrist added

File: assignment4/urdf/lynxmotion.urdf (robot description, URDF)
Before this commit: robot lynxmotion, 4 links, 3 joints
Links:
- removed link base_block
- added link base_rotate; visual cylinder length=0.2 radius=0.1
- added link left_gripper; visual mesh filename=package://urdf_tutorial/meshes/l_finger.dae
- added link right_gripper; visual mesh filename=package://urdf_tutorial/meshes/l_finger.dae
- added link wrist; visual box size=0.2 0.1 0.05
- link base_link: geometry visual cylinder length=0.2 radius=0.3
- link bottom_arm: geometry visual box size=0.4 0.2 0.05
- link top_arm: geometry visual box size=0.4 0.2 0.05
Joints:
- added joint left_gripper_joint: type revolute, parent wrist, child left_gripper, origin xyz=0 0 0.2 rpy=0 0 0, axis 0 1 0, limit lower=-1.57075 upper=0 effort=1000.0 velocity=0.5
- added joint right_gripper_joint: type revolute, parent wrist, child right_gripper, origin xyz=0 0 0.2 rpy=0 0 0, axis 0 0 -1, limit lower=0.0 upper=0.548 effort=1000.0 velocity=0.5
- added joint wrist_rotate: type revolute, parent top_arm, child wrist, origin xyz=0 0 0.4, axis 0 0 1, limit lower=-1.548 upper=1.548 effort=1000.0 velocity=0.5
- joint base_block_to_base_link: child base_link -> base_rotate; origin xyz=0 0 0.4 -> xyz=0 0 0.1; parent base_block -> base_link
- joint base_to_bottom_arm: origin xyz=0 0 0.5 -> xyz=0 0 0.2; parent base_link -> base_rotate
- joint bottom_to_top_arm: origin xyz=0 0 0.3 -> xyz=0 0 0.4

File: assignment4/urdf/lynxmotion.urdf.xacro (robot description, xacro)
@@ -4,18 +4,21 @@
 		<color rgba="0 0 0.8 1"/>
 	</material>
-	<link name="base_block">
+	<material name="green">
+		<color rgba="0 0.5 0 1"/>
+	</material>
+	<link name="base_link">
 		<visual>
 			<geometry>
 				<cylinder length="0.2" radius="0.3"/>
 			</geometry>
-			<origin rpy="0 0 0" xyz="0 0 0.3"/>
+			<material name="green"/>
 		</visual>
 	</link>
-	<link name="base_link">
+	<link name="base_rotate">
 		<visual>
 			<geometry>
 				<cylinder length="0.2" radius="0.1"/>
 			</geometry>
-			<origin rpy="0 0 0" xyz="0 0 0.3"/>
+			<origin rpy="0 0 0" xyz="0 0 0.1"/>
 		</visual>
 	</link>
@@ -23,8 +26,8 @@
 		<visual>
 			<geometry>
-				<box size="0.4 0.1 0.2"/>
+				<box size="0.4 0.2 0.05"/>
 			</geometry>
 			<material name="blue"/>
-			<origin rpy="0 1.57075 0" xyz="0 0 0.15"/>
+			<origin rpy="0 1.57075 0" xyz="0 0 0.2"/>
 		</visual>
 	</link>
@@ -32,21 +35,59 @@
 		<visual>
 			<geometry>
-				<box size="0.4 0.1 0.2"/>
+				<box size="0.4 0.2 0.05"/>
 			</geometry>
-			<origin rpy="0 1.57075 0" xyz="0 0 0.3"/>
+			<origin rpy="0 1.57075 0" xyz="0 0 0.2"/>
 		</visual>
 	</link>
+	<link name="wrist">
+		<visual>
+			<geometry>
+				<box size="0.2 0.1 0.05"/>
+			</geometry>
+			<origin rpy="0 -1.57075 0" xyz="0 0 0.1"/>
+		</visual>
+	</link>
+	<link name="right_gripper">
+		<visual>
+			<origin rpy="-1.57075 1.57075 0" xyz="0 0 0"/>
+			<geometry>
+				<mesh filename="package://urdf_tutorial/meshes/l_finger.dae"/>
+			</geometry>
+		</visual>
+	</link>
+	<link name="left_gripper">
+		<visual>
+			<origin rpy="1.57075 -1.57075 3.1415" xyz="0 0 0"/>
+			<geometry>
+				<mesh filename="package://urdf_tutorial/meshes/l_finger.dae"/>
+			</geometry>
+		</visual>
+	</link>
+	<joint name="left_gripper_joint" type="revolute">
+		<axis xyz="0 1 0"/>
+		<limit effort="1000.0" lower="-1.57075" upper="0" velocity="0.5"/>
+		<origin rpy="0 0 0" xyz="0 0 0.2"/>
+		<parent link="wrist"/>
+		<child link="left_gripper"/>
+	</joint>
+	<joint name="right_gripper_joint" type="revolute">
+		<axis xyz="0 0 -1"/>
+		<limit effort="1000.0" lower="0.0" upper="0.548" velocity="0.5"/>
+		<origin rpy="0 0 0" xyz="0 0 0.2"/>
+		<parent link="wrist"/>
+		<child link="right_gripper"/>
+	</joint>
 	<joint name="base_block_to_base_link" type="revolute">
 		<axis xyz="0 0 1"/>
 		<limit effort="1000.0" lower="-1.548" upper="1.548" velocity="0.5"/>
-		<origin xyz="0 0 0.4"/>
-		<parent link="base_block"/>
-		<child link="base_link"/>
+		<origin xyz="0 0 0.1"/>
+		<parent link="base_link"/>
+		<child link="base_rotate"/>
 	</joint>
 	<joint name="base_to_bottom_arm" type="revolute">
 		<axis xyz="0 1 0"/>
 		<limit effort="1000.0" lower="-1.548" upper="1.548" velocity="0.5"/>
-		<origin xyz="0 0 0.5"/>
-		<parent link="base_link"/>
+		<origin xyz="0 0 0.2"/>
+		<parent link="base_rotate"/>
 		<child link="bottom_arm"/>
 	</joint>
@@ -54,7 +95,14 @@
 		<axis xyz="0 1 0"/>
 		<limit effort="1000.0" lower="-1.548" upper="1.548" velocity="0.5"/>
-		<origin xyz="0 0 0.3"/>
+		<origin xyz="0 0 0.4"/>
 		<parent link="bottom_arm"/>
 		<child link="top_arm"/>
 	</joint>
+	<joint name="wrist_rotate" type="revolute">
+		<axis xyz="0 0 1"/>
+		<limit effort="1000.0" lower="-1.548" upper="1.548" velocity="0.5"/>
+		<origin xyz="0 0 0.4"/>
+		<parent link="top_arm"/>
+		<child link="wrist"/>
+	</joint>
 </robot>

Commit message: fixed gripper positions

File: assignment4/urdf/lynxmotion.urdf (robot description, URDF)
Before this commit: robot lynxmotion, 7 links, 6 joints
Joints:
- joint left_gripper_joint: limit lower=-1.57075 upper=0 effort=1000.0 velocity=0.5 -> lower=0 upper=1.57075 effort=1000.0 velocity=0.5
- joint right_gripper_joint: axis 0 0 -1 -> 0 1 0; limit lower=0.0 upper=0.548 effort=1000.0 velocity=0.5 -> lower=-1.57075 upper=0 effort=1000.0 velocity=0.5

File: assignment4/urdf/lynxmotion.urdf.xacro (robot description, xacro)
@@ -6,4 +6,7 @@
 	<material name="green">
 		<color rgba="0 0.5 0 1"/>
+	</material>
+	<material name="light_blue">
+		<color rgba="0 0.25 0.5 1"/>
 	</material>
 	<link name="base_link">
@@ -50,21 +53,23 @@
 	<link name="right_gripper">
 		<visual>
-			<origin rpy="-1.57075 1.57075 0" xyz="0 0 0"/>
+			<origin rpy="-1.57075 0 0" xyz="0 0 0"/>
 			<geometry>
 				<mesh filename="package://urdf_tutorial/meshes/l_finger.dae"/>
 			</geometry>
+			<material name="light_blue"/>
 		</visual>
 	</link>
 	<link name="left_gripper">
 		<visual>
-			<origin rpy="1.57075 -1.57075 3.1415" xyz="0 0 0"/>
+			<origin rpy="-1.57075 0 3.1415" xyz="0 0 0"/>
 			<geometry>
 				<mesh filename="package://urdf_tutorial/meshes/l_finger.dae"/>
 			</geometry>
+			<material name="light_blue"/>
 		</visual>
 	</link>
 	<joint name="left_gripper_joint" type="revolute">
 		<axis xyz="0 1 0"/>
-		<limit effort="1000.0" lower="-1.57075" upper="0" velocity="0.5"/>
+		<limit effort="1000.0" lower="0" upper="1.57075" velocity="0.5"/>
 		<origin rpy="0 0 0" xyz="0 0 0.2"/>
 		<parent link="wrist"/>
@@ -72,6 +77,6 @@
 	</joint>
 	<joint name="right_gripper_joint" type="revolute">
-		<axis xyz="0 0 -1"/>
-		<limit effort="1000.0" lower="0.0" upper="0.548" velocity="0.5"/>
+		<axis xyz="0 1 0"/>
+		<limit effort="1000.0" lower="-1.57075" upper="0" velocity="0.5"/>
 		<origin rpy="0 0 0" xyz="0 0 0.2"/>
 		<parent link="wrist"/>

Commit message: added 3rd deg of freedom

File: assignment4/urdf/lynxmotion.urdf (robot description, URDF)
Before this commit: robot lynxmotion, 7 links, 6 joints
Links:
- added link fore_arm; visual box size=0.1 0.1 0.05
- link wrist: geometry visual box size=0.1 0.1 0.05
Joints:
- added joint top_to_fore_arm: type revolute, parent top_arm, child fore_arm, origin xyz=0 0 0.4, axis 0 1 0, limit lower=-1.548 upper=1.548 effort=1000.0 velocity=0.5
- joint left_gripper_joint: origin xyz=0 0 0.2 rpy=0 0 0 -> xyz=0 0 0.1 rpy=0 0 0
- joint right_gripper_joint: origin xyz=0 0 0.2 rpy=0 0 0 -> xyz=0 0 0.1 rpy=0 0 0
- joint wrist_rotate: origin xyz=0 0 0.4 -> xyz=0 0 0.1; parent top_arm -> fore_arm

File: assignment4/urdf/lynxmotion.urdf.xacro (robot description, xacro)
@@ -43,10 +43,19 @@
 		</visual>
 	</link>
+	<link name="fore_arm">
+		<visual>
+			<geometry>
+				<box size="0.1 0.1 0.05"/>
+			</geometry>
+			<material name="light_blue"/>
+			<origin rpy="0 1.57075 0" xyz="0 0 0.05"/>
+		</visual>
+	</link>
 	<link name="wrist">
 		<visual>
 			<geometry>
-				<box size="0.2 0.1 0.05"/>
+				<box size="0.1 0.1 0.05"/>
 			</geometry>
-			<origin rpy="0 -1.57075 0" xyz="0 0 0.1"/>
+			<origin rpy="0 -1.57075 0" xyz="0 0 0.05"/>
 		</visual>
 	</link>
@@ -72,5 +81,5 @@
 		<axis xyz="0 1 0"/>
 		<limit effort="1000.0" lower="0" upper="1.57075" velocity="0.5"/>
-		<origin rpy="0 0 0" xyz="0 0 0.2"/>
+		<origin rpy="0 0 0" xyz="0 0 0.1"/>
 		<parent link="wrist"/>
 		<child link="left_gripper"/>
@@ -79,5 +88,5 @@
 		<axis xyz="0 1 0"/>
 		<limit effort="1000.0" lower="-1.57075" upper="0" velocity="0.5"/>
-		<origin rpy="0 0 0" xyz="0 0 0.2"/>
+		<origin rpy="0 0 0" xyz="0 0 0.1"/>
 		<parent link="wrist"/>
 		<child link="right_gripper"/>
@@ -104,9 +113,16 @@
 		<child link="top_arm"/>
 	</joint>
+	<joint name="top_to_fore_arm" type="revolute">
+		<axis xyz="0 1 0"/>
+		<limit effort="1000.0" lower="-1.548" upper="1.548" velocity="0.5"/>
+		<origin xyz="0 0 0.4"/>
+		<parent link="top_arm"/>
+		<child link="fore_arm"/>
+	</joint>
 	<joint name="wrist_rotate" type="revolute">
 		<axis xyz="0 0 1"/>
 		<limit effort="1000.0" lower="-1.548" upper="1.548" velocity="0.5"/>
-		<origin xyz="0 0 0.4"/>
-		<parent link="top_arm"/>
+		<origin xyz="0 0 0.1"/>
+		<parent link="fore_arm"/>
 		<child link="wrist"/>
 	</joint>

Commit message: change thickness of limbs

File: assignment4/urdf/lynxmotion.urdf (robot description, URDF)
Before this commit: robot lynxmotion, 8 links, 7 joints
Links:
- link bottom_arm: geometry visual box size=0.4 0.1 0.05
- link top_arm: geometry visual box size=0.4 0.1 0.05

File: assignment4/urdf/lynxmotion.urdf.xacro (robot description, xacro)
@@ -29,5 +29,5 @@
 		<visual>
 			<geometry>
-				<box size="0.4 0.2 0.05"/>
+				<box size="0.4 0.1 0.05"/>
 			</geometry>
 			<material name="blue"/>
@@ -38,5 +38,5 @@
 		<visual>
 			<geometry>
-				<box size="0.4 0.2 0.05"/>
+				<box size="0.4 0.1 0.05"/>
 			</geometry>
 			<origin rpy="0 1.57075 0" xyz="0 0 0.2"/>
